Commit message: feat: move lidar link to config

File: config/ego_racecar.xacro (robot description, xacro)
@@ -18,4 +18,6 @@
     <color rgba="1.0 0. 0. 1."/>
   </material>
+  <!-- ${car_name}/laser is NOT a joint here: the real laser pose comes from
+       stack_master/config/<racecar_version>/static_transforms.yaml (static_transforms_launch.xml). -->
   <link name="${car_name}/base_link">
     <visual>
@@ -26,12 +28,6 @@
       <material name="blue"/>
     </visual>
-  </link>
-  <joint name="base_to_laser" type="fixed">
-    <parent link="${car_name}/base_link"/>
-    <child link="${car_name}/laser"/>
-    <origin xyz="${laser_distance_from_base_link} 0 ${ground_offset+height+(laser_height/2)}"/>
-  </joint>
-  <link name="${car_name}/laser">
     <visual>
+      <origin xyz="${laser_distance_from_base_link} 0 ${ground_offset+height+(laser_height/2)}"/>
       <geometry>
         <cylinder radius="${laser_radius}" length="${laser_height}"/>
